Commit message: Add files via upload

File: ros_mm_arm_description/urdf/ros_mm_arm.urdf (robot description, URDF)
Before this commit: robot ros_mm_arm, 16 links, 15 joints
Links:
- link arm_elbow_F3_0_link: geometry collision box size=0.025 0.038 0.009; visual mesh filename=package://ros_mm_arm_description/meshes/F3.stl scale=0.001 0.001 0.001
- link arm_shoulder_lift_link: geometry collision box size=0.028 0.0485 0.065; visual mesh filename=package://ros_mm_arm_description/meshes/F4.stl scale=0.001 0.001 0.001
- link arm_shoulder_lift_servo_link: geometry collision box size=0.025 0.038 0.04762; visual mesh filename=package://ros_mm_arm_description/meshes/ax12_box.stl scale=0.001 0.001 0.001
- link arm_shoulder_pan_link: geometry collision box size=0.025 0.038 0.009; visual mesh filename=package://ros_mm_arm_description/meshes/F3.stl scale=0.001 0.001 0.001
- link arm_shoulder_pan_servo_link: geometry collision box size=0.025 0.038 0.04762; visual mesh filename=package://ros_mm_arm_description/meshes/ax12_box.stl scale=0.001 0.001 0.001
- link arm_wrist_F3_0_link: geometry collision box size=0.025 0.038 0.009; visual mesh filename=package://ros_mm_arm_description/meshes/F3.stl scale=0.001 0.001 0.001
- link arm_wrist_flex_link: geometry collision box size=0.025 0.0485 0.0375; visual mesh filename=package://ros_mm_arm_description/meshes/F2.stl scale=0.001 0.001 0.001
- link arm_wrist_flex_servo_link: geometry collision box size=0.025 0.038 0.04762; visual mesh filename=package://ros_mm_arm_description/meshes/ax12_box.stl scale=0.001 0.001 0.001
- link gripper_active_finger_link: geometry collision box size=0.0783 0.03801 0.0193; visual mesh filename=package://ros_mm_arm_description/meshes/turtlebot_finger.stl scale=0.001 0.001 0.001
- link gripper_active_link: geometry collision box size=0.025 0.0485 0.0375; visual mesh filename=package://ros_mm_arm_description/meshes/F2.stl scale=0.001 0.001 0.001
- link gripper_servo_link: geometry collision box size=0.025 0.038 0.04762; visual mesh filename=package://ros_mm_arm_description/meshes/ax12_box.stl scale=0.001 0.001 0.001
- link gripper_static_finger_link: geometry collision box size=0.0783 0.03801 0.0193; visual mesh filename=package://ros_mm_arm_description/meshes/turtlebot_finger.stl scale=0.001 0.001 0.001
- link gripper_static_link: geometry collision box size=0.025 0.038 0.009; visual mesh filename=package://ros_mm_arm_description/meshes/F3.stl scale=0.001 0.001 0.001

File: ros_mm_arm_description/urdf/ros_mm_arm_2.urdf (robot description, URDF)
Before this commit: robot ros_mm_arm_2, 16 links, 15 joints
Links:
- link arm_elbow_F3_0_link: geometry collision box size=0.025 0.038 0.009; visual mesh filename=package://ros_mm_arm_description/meshes/F3.stl scale=0.001 0.001 0.001
- link arm_shoulder_lift_link: geometry collision box size=0.028 0.0485 0.065; visual mesh filename=package://ros_mm_arm_description/meshes/F4.stl scale=0.001 0.001 0.001
- link arm_shoulder_lift_servo_link: geometry collision box size=0.025 0.038 0.04762; visual mesh filename=package://ros_mm_arm_description/meshes/ax12_box.stl scale=0.001 0.001 0.001
- link arm_shoulder_pan_link: geometry collision box size=0.025 0.038 0.009; visual mesh filename=package://ros_mm_arm_description/meshes/F3.stl scale=0.001 0.001 0.001
- link arm_shoulder_pan_servo_link: geometry collision box size=0.025 0.038 0.04762; visual mesh filename=package://ros_mm_arm_description/meshes/ax12_box.stl scale=0.001 0.001 0.001
- link arm_wrist_F3_0_link: geometry collision box size=0.025 0.038 0.009; visual mesh filename=package://ros_mm_arm_description/meshes/F3.stl scale=0.001 0.001 0.001
- link arm_wrist_flex_link: geometry collision box size=0.025 0.0485 0.0375; visual mesh filename=package://ros_mm_arm_description/meshes/F2.stl scale=0.001 0.001 0.001
- link arm_wrist_flex_servo_link: geometry collision box size=0.025 0.038 0.04762; visual mesh filename=package://ros_mm_arm_description/meshes/ax12_box.stl scale=0.001 0.001 0.001
- link gripper_active_finger_link: geometry collision box size=0.0783 0.03801 0.0193; visual mesh filename=package://ros_mm_arm_description/meshes/turtlebot_finger.stl scale=0.001 0.001 0.001
- link gripper_active_link: geometry collision box size=0.025 0.0485 0.0375; visual mesh filename=package://ros_mm_arm_description/meshes/F2.stl scale=0.001 0.001 0.001
- link gripper_servo_link: geometry collision box size=0.025 0.038 0.04762; visual mesh filename=package://ros_mm_arm_description/meshes/ax12_box.stl scale=0.001 0.001 0.001
- link gripper_static_finger_link: geometry collision box size=0.0783 0.03801 0.0193; visual mesh filename=package://ros_mm_arm_description/meshes/turtlebot_finger.stl scale=0.001 0.001 0.001
- link gripper_static_link: geometry collision box size=0.025 0.038 0.009; visual mesh filename=package://ros_mm_arm_description/meshes/F3.stl scale=0.001 0.001 0.001
